Commit message: fix bugs

File: palletizer_model_pkg/urdf/palletizer_model.urdf (robot description, URDF)
Before this commit: robot palletizer_model, 13 links, 12 joints
Joints:
- joint pal_base: origin xyz=0 0 0 rpy=0 0 -1.57 -> xyz=0 0 0.05 rpy=0 0 -1.57

File: vertical_robot_model/urdf/vertical_robot.urdf (robot description, URDF)
Before this commit: robot vertical_robot, 8 links, 7 joints
Joints:
- joint world_joint: origin (none) -> xyz=0.0 0.0 0.0 rpy=0 0 0
