Commit message: scale model

File: palletizer_model_pkg/urdf/palletizer_model.urdf.xacro (robot description, xacro)
@@ -1,4 +1,5 @@
 <?xml version="1.0" ?>
 <robot name="palletizer_model" xmlns:xacro="http://www.ros.org/wiki/xacro">
+	<xacro:include filename="$(find palletizer_model_pkg)/urdf/config.xacro" />
 	<link name ="world"/>
 	<joint name="pal_base" type="fixed">
@@ -12,10 +13,10 @@
 			<origin xyz = "0 0 0" rpy="0 0 0" />
 			<geometry>
-				<mesh filename="package://palletizer_model_pkg/meshes/link0.stl" scale="0.001 0.001 0.001"/>
-			</geometry>
-		</collision>
-		<visual>
-			<geometry>
-				<mesh filename="package://palletizer_model_pkg/meshes/link0.stl" scale="0.001 0.001 0.001"/>
+				<mesh filename="package://palletizer_model_pkg/meshes/link0.stl" scale="${scale_param*0.001} ${scale_param*0.001} ${scale_param*0.001}"/>
+			</geometry>
+		</collision>
+		<visual>
+			<geometry>
+				<mesh filename="package://palletizer_model_pkg/meshes/link0.stl" scale="${scale_param*0.001} ${scale_param*0.001} ${scale_param*0.001}"/>
 			</geometry>
 			<material name="grey">
@@ -27,5 +28,5 @@
 		<parent link="pal_link0"/>
 		<child link="pal_link1"/>
-		<origin xyz = "0 0 0.107" rpy="0 0 1.57" />
+		<origin xyz = "0 0 ${scale_param*0.107}" rpy="0 0 1.57" />
 		<axis xyz="0 0 1" />
 	</joint>
@@ -34,10 +35,10 @@
 			<origin xyz = "0 0 0" rpy="0 0 0" />
 			<geometry>
-				<mesh filename="package://palletizer_model_pkg/meshes/link1.stl" scale="0.001 0.001 0.001"/>
-			</geometry>
-		</collision>
-		<visual>
-			<geometry>
-				<mesh filename="package://palletizer_model_pkg/meshes/link1.stl" scale="0.001 0.001 0.001"/>
+				<mesh filename="package://palletizer_model_pkg/meshes/link1.stl" scale="${scale_param*0.001} ${scale_param*0.001} ${scale_param*0.001}"/>
+			</geometry>
+		</collision>
+		<visual>
+			<geometry>
+				<mesh filename="package://palletizer_model_pkg/meshes/link1.stl" scale="${scale_param*0.001} ${scale_param*0.001} ${scale_param*0.001}"/>
 			</geometry>
 			<material name="grey">
@@ -49,5 +50,5 @@
 		<parent link="pal_link1"/>
 		<child link="pal_link2"/>
-		<origin xyz = "-0.0065 -0.021131 0.04662" rpy="0 -1.57 0" />
+		<origin xyz = "${-0.0065*scale_param} ${-0.021131*scale_param} ${0.04662*scale_param}" rpy="0 -1.57 0" />
 		<axis xyz="0 0 -1" />
 		<limit effort="1.0" lower="-1.57" upper="1.57" velocity="5.0"/>
@@ -57,10 +58,10 @@
 			<origin xyz = "0 0 0" rpy="0 0 0" />
 			<geometry>
-				<mesh filename="package://palletizer_model_pkg/meshes/link2.stl" scale="0.001 0.001 0.001"/>
-			</geometry>
-		</collision>
-		<visual>
-			<geometry>
-				<mesh filename="package://palletizer_model_pkg/meshes/link2.stl" scale="0.001 0.001 0.001"/>
+				<mesh filename="package://palletizer_model_pkg/meshes/link2.stl" scale="${scale_param*0.001} ${scale_param*0.001} ${scale_param*0.001}"/>
+			</geometry>
+		</collision>
+		<visual>
+			<geometry>
+				<mesh filename="package://palletizer_model_pkg/meshes/link2.stl" scale="${scale_param*0.001} ${scale_param*0.001} ${scale_param*0.001}"/>
 			</geometry>
 			<material name="grey">
@@ -72,5 +73,5 @@
 		<parent link="pal_link1"/>
 		<child link="pal_link8"/>
-		<origin xyz = "0.0065 -0.02113 0.04636" rpy="0 0 0" />
+		<origin xyz = "${0.0065*scale_param} ${-0.02113*scale_param} ${0.04636*scale_param}" rpy="0 0 0" />
 		<axis xyz="-1 0 0" />
 		<limit effort="1.0" lower="-1.57" upper="1.57" velocity="5.0"/>
@@ -80,10 +81,10 @@
 			<origin xyz = "0 0 0" rpy="0 0 0" />
 			<geometry>
-				<mesh filename="package://palletizer_model_pkg/meshes/link3.stl" scale="0.001 0.001 0.001"/>
-			</geometry>
-		</collision>
-		<visual>
-			<geometry>
-				<mesh filename="package://palletizer_model_pkg/meshes/link3.stl" scale="0.001 0.001 0.001"/>
+				<mesh filename="package://palletizer_model_pkg/meshes/link3.stl" scale="${scale_param*0.001} ${scale_param*0.001} ${scale_param*0.001}"/>
+			</geometry>
+		</collision>
+		<visual>
+			<geometry>
+				<mesh filename="package://palletizer_model_pkg/meshes/link3.stl" scale="${scale_param*0.001} ${scale_param*0.001} ${scale_param*0.001}"/>
 			</geometry>
 			<material name="grey">
@@ -96,10 +97,10 @@
 			<origin xyz = "0 0 0" rpy="0 0 0" />
 			<geometry>
-				<mesh filename="package://palletizer_model_pkg/meshes/link4.stl" scale="0.001 0.001 0.001"/>
-			</geometry>
-		</collision>
-		<visual>
-			<geometry>
-				<mesh filename="package://palletizer_model_pkg/meshes/link4.stl" scale="0.001 0.001 0.001"/>
+				<mesh filename="package://palletizer_model_pkg/meshes/link4.stl" scale="${scale_param*0.001} ${scale_param*0.001} ${scale_param*0.001}"/>
+			</geometry>
+		</collision>
+		<visual>
+			<geometry>
+				<mesh filename="package://palletizer_model_pkg/meshes/link4.stl" scale="${scale_param*0.001} ${scale_param*0.001} ${scale_param*0.001}"/>
 			</geometry>
 			<material name="grey">
@@ -111,5 +112,5 @@
 		<parent link="pal_link4"/>
 		<child link="pal_link4_1"/>
-		<origin xyz = "0 -0.0495 -0.017" rpy="0 0 0" />
+		<origin xyz = "0 ${-0.0495*scale_param} ${-0.017*scale_param}" rpy="0 0 0" />
 		<axis xyz="0 0 -1" />
 		<limit effort="1.0" lower="-3.14" upper="3.14" velocity="5.0"/>
@@ -119,10 +120,10 @@
 			<origin xyz = "0 0 0" rpy="0 0 0" />
 			<geometry>
-				<mesh filename="package://palletizer_model_pkg/meshes/link4_1.stl" scale="0.001 0.001 0.001"/>
-			</geometry>
-		</collision>
-		<visual>
-			<geometry>
-				<mesh filename="package://palletizer_model_pkg/meshes/link4_1.stl" scale="0.001 0.001 0.001"/>
+				<mesh filename="package://palletizer_model_pkg/meshes/link4_1.stl" scale="${scale_param*0.001} ${scale_param*0.001} ${scale_param*0.001}"/>
+			</geometry>
+		</collision>
+		<visual>
+			<geometry>
+				<mesh filename="package://palletizer_model_pkg/meshes/link4_1.stl" scale="${scale_param*0.001} ${scale_param*0.001} ${scale_param*0.001}"/>
 			</geometry>
 			<material name="grey">
@@ -134,5 +135,5 @@
 		<parent link="pal_link4_1"/>
 		<child link="prisos"/>
-		<origin xyz = "0.001 -0.041 -0.066" rpy="0 0 -1.57" />
+		<origin xyz = "${0.001*scale_param} ${-0.041*scale_param} ${-0.066*scale_param}" rpy="0 0 -1.57" />
 	</joint>
 	<link name="prisos">
@@ -140,10 +141,10 @@
 			<origin xyz = "0 0 0" rpy="0 0 0" />
 			<geometry>
-				<mesh filename="package://palletizer_model_pkg/meshes/prisos.stl" scale="0.001 0.001 0.001"/>
-			</geometry>
-		</collision>
-		<visual>
-			<geometry>
-				<mesh filename="package://palletizer_model_pkg/meshes/prisos.stl" scale="0.001 0.001 0.001"/>
+				<mesh filename="package://palletizer_model_pkg/meshes/prisos.stl" scale="${scale_param*0.001} ${scale_param*0.001} ${scale_param*0.001}"/>
+			</geometry>
+		</collision>
+		<visual>
+			<geometry>
+				<mesh filename="package://palletizer_model_pkg/meshes/prisos.stl" scale="${scale_param*0.001} ${scale_param*0.001} ${scale_param*0.001}"/>
 			</geometry>
 			<material name="grey">
@@ -155,5 +156,5 @@
 		<parent link="pal_link3"/>
 		<child link="pal_link4"/>
-		<origin xyz = "-0.160 0 0" rpy="-1.57 -1.57 0" />
+		<origin xyz = "${-0.160*scale_param} 0 0" rpy="-1.57 -1.57 0" />
 		<axis xyz="1 0 0" />
 		<mimic joint="pal_joint1" multiplier="-1" offset="0"/>
@@ -162,5 +163,5 @@
 		<parent link="pal_link1"/>
 		<child link="pal_link5"/>
-		<origin xyz = "0.0339 0.01328 0.070418" rpy="1.57 0 3.14" />
+		<origin xyz = "${0.0339*scale_param} ${0.01328*scale_param} ${0.070418*scale_param}" rpy="1.57 0 3.14" />
 		<axis xyz="1 0 0" />
 		<mimic joint="pal_joint1" multiplier="1" offset="0"/>
@@ -170,10 +171,10 @@
 			<origin xyz = "0 0 0" rpy="0 0 0" />
 			<geometry>
-				<mesh filename="package://palletizer_model_pkg/meshes/link5.stl" scale="0.001 0.001 0.001"/>
-			</geometry>
-		</collision>
-		<visual>
-			<geometry>
-				<mesh filename="package://palletizer_model_pkg/meshes/link5.stl" scale="0.001 0.001 0.001"/>
+				<mesh filename="package://palletizer_model_pkg/meshes/link5.stl" scale="${scale_param*0.001} ${scale_param*0.001} ${scale_param*0.001}"/>
+			</geometry>
+		</collision>
+		<visual>
+			<geometry>
+				<mesh filename="package://palletizer_model_pkg/meshes/link5.stl" scale="${scale_param*0.001} ${scale_param*0.001} ${scale_param*0.001}"/>
 			</geometry>
 			<material name="grey">
@@ -185,5 +186,5 @@
 		<parent link="pal_link2"/>
 		<child link="pal_link6"/>
-		<origin xyz = "0.148 0 -0.0205" rpy="0 0 0" />
+		<origin xyz = "${0.148*scale_param} 0 ${-0.0205*scale_param}" rpy="0 0 0" />
 		<axis xyz="0 0 1" />
 		<mimic joint="pal_joint3" multiplier="-1" offset="0"/>
@@ -193,10 +194,10 @@
 			<origin xyz = "0 0 0" rpy="0 0 0" />
 			<geometry>
-				<mesh filename="package://palletizer_model_pkg/meshes/link6.stl" scale="0.001 0.001 0.001"/>
-			</geometry>
-		</collision>
-		<visual>
-			<geometry>
-				<mesh filename="package://palletizer_model_pkg/meshes/link6.stl" scale="0.001 0.001 0.001"/>
+				<mesh filename="package://palletizer_model_pkg/meshes/link6.stl" scale="${scale_param*0.001} ${scale_param*0.001} ${scale_param*0.001}"/>
+			</geometry>
+		</collision>
+		<visual>
+			<geometry>
+				<mesh filename="package://palletizer_model_pkg/meshes/link6.stl" scale="${scale_param*0.001} ${scale_param*0.001} ${scale_param*0.001}"/>
 			</geometry>
 			<material name="grey">
@@ -208,5 +209,5 @@
 		<parent link="pal_link4"/>
 		<child link="pal_link7"/>
-		<origin xyz = "0.024 -0.034404 0.02409" rpy="3.14 0 0" />
+		<origin xyz = "${0.024*scale_param} ${-0.034404*scale_param} ${0.02409*scale_param}" rpy="3.14 0 0" />
 		<axis xyz="1 0 0" />
 		<mimic joint="pal_joint3" multiplier="-1" offset="0"/>
@@ -216,10 +217,10 @@
 			<origin xyz = "0 0 0" rpy="0 0 0" />
 			<geometry>
-				<mesh filename="package://palletizer_model_pkg/meshes/link7.stl" scale="0.001 0.001 0.001"/>
-			</geometry>
-		</collision>
-		<visual>
-			<geometry>
-				<mesh filename="package://palletizer_model_pkg/meshes/link7.stl" scale="0.001 0.001 0.001"/>
+				<mesh filename="package://palletizer_model_pkg/meshes/link7.stl" scale="${scale_param*0.001} ${scale_param*0.001} ${scale_param*0.001}"/>
+			</geometry>
+		</collision>
+		<visual>
+			<geometry>
+				<mesh filename="package://palletizer_model_pkg/meshes/link7.stl" scale="${scale_param*0.001} ${scale_param*0.001} ${scale_param*0.001}"/>
 			</geometry>
 			<material name="grey">
@@ -231,5 +232,5 @@
 		<parent link="pal_link2"/>
 		<child link="pal_link3"/>
-		<origin xyz = "0.148 0 0" rpy="0 3.14 -1.57" />
+		<origin xyz = "${0.148*scale_param} 0 0" rpy="0 3.14 -1.57" />
 		<axis xyz="0 0 1" />
 		<mimic joint="pal_joint2" multiplier="1" offset="0"/>
@@ -239,10 +240,10 @@
 			<origin xyz = "0 0 0" rpy="0 0 0" />
 			<geometry>
-				<mesh filename="package://palletizer_model_pkg/meshes/link8.stl" scale="0.001 0.001 0.001"/>
-			</geometry>
-		</collision>
-		<visual>
-			<geometry>
-				<mesh filename="package://palletizer_model_pkg/meshes/link8.stl" scale="0.001 0.001 0.001"/>
+				<mesh filename="package://palletizer_model_pkg/meshes/link8.stl" scale="${scale_param*0.001} ${scale_param*0.001} ${scale_param*0.001}"/>
+			</geometry>
+		</collision>
+		<visual>
+			<geometry>
+				<mesh filename="package://palletizer_model_pkg/meshes/link8.stl" scale="${scale_param*0.001} ${scale_param*0.001} ${scale_param*0.001}"/>
 			</geometry>
 			<material name="grey">
@@ -254,5 +255,5 @@
 		<parent link="pal_link8"/>
 		<child link="pal_link9"/>
-		<origin xyz = "-0.021 0.054 0" rpy="1.57 0 0" />
+		<origin xyz = "${-0.021*scale_param} ${0.054*scale_param} 0" rpy="1.57 0 0" />
 		<axis xyz="1 0 0" />
 		<mimic joint="pal_joint1" multiplier="-1" offset="0"/>
@@ -262,10 +263,10 @@
 			<origin xyz = "0 0 0" rpy="0 0 0" />
 			<geometry>
-				<mesh filename="package://palletizer_model_pkg/meshes/link9.stl" scale="0.001 0.001 0.001"/>
-			</geometry>
-		</collision>
-		<visual>
-			<geometry>
-				<mesh filename="package://palletizer_model_pkg/meshes/link9.stl" scale="0.001 0.001 0.001"/>
+				<mesh filename="package://palletizer_model_pkg/meshes/link9.stl" scale="${scale_param*0.001} ${scale_param*0.001} ${scale_param*0.001}"/>
+			</geometry>
+		</collision>
+		<visual>
+			<geometry>
+				<mesh filename="package://palletizer_model_pkg/meshes/link9.stl" scale="${scale_param*0.001} ${scale_param*0.001} ${scale_param*0.001}"/>
 			</geometry>
 			<material name="grey">
