Commit message: controller

File: palletizer_model_pkg/urdf/config.xacro (robot description, xacro)
@@ -1,4 +1,4 @@
 <?xml version="1.0" ?>
 <robot xmlns:xacro="http://www.ros.org/wiki/xacro">
-  <xacro:property name="scale_param" value="1" />
+  <xacro:property name="scale_param" value="1.5" />
 </robot>
